File: Engine_monitor_V1/Engine_monitor_V1.kicad_pcb (KiCad board)
At the start: 2 copper layers, 50.6 x 75.1 mm, 36 parts, among them J1 RPM_PICKUP, J2 Screw_Terminal_01x02, U1 nice_nano, U2 LMV331, U3 MAX31856, U4 MAX31856, X1 3.5mm term, X2 3.5mm term

Commit message: Update the schematic
RPM meter isn't working, swapped a cap for a resistor.
Parts:
- removed C7: 10nF, Capacitor_SMD:C_0805_2012Metric
- added R14: 220k, Resistor_SMD:R_0805_2012Metric, F.Cu at (97.7, 82.5)
Changed lines of the file:
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@@
 		)
 	)
-	(footprint "Capacitor_SMD:C_0805_2012Metric"
-		(layer "F.Cu")
-		(at 97.75 82.45)
-		(descr "Capacitor SMD 0805 (2012 Metric), square (rectangular) end terminal, IPC-7351 nominal, (Body size source: IPC-SM-782 page 76, https://www.pcb-3d.com/wordpress/wp-content/uploads/ipc-sm-782a_amendment_1_and_2.pdf, https://docs.google.com/spreadsheets/d/1BsfQQcO9C6DZCsRaXUlFlo91Tg2WpOkGARC1WS5S8t0/edit?usp=sharing)")
-		(tags "capacitor")
-		(property "Reference" "C7"
-			(at 3.75 2.05 0)
-			(layer "F.SilkS")
-			(effects
-				(font
-					(size 0.6 0.6)
-					(thickness 0.1)
-					(bold yes)
-				)
-			)
-		)
-		(property "Value" "10nF"
-			(at 4.05 0.1 0)
-			(layer "F.Fab")
-			(effects
-				(font
-					(size 0.6 0.6)
-					(thickness 0.1)
-					(bold yes)
-				)
-			)
-		)
-		(property "Datasheet" ""
-			(at 0 0 0)
-			(layer "F.Fab")
-			(hide yes)
-			(effects
-				(font
-					(size 1.27 1.27)
-				)
-			)
-		)
-		(property "Description" "Unpolarized capacitor"
-			(at 0 0 0)
-			(layer "F.Fab")
-			(hide yes)
-			(effects
-				(font
-					(size 1.27 1.27)
-				)
-			)
-		)
-		(property "KiLib_Generator" "SMD_2terminal_chip_molded"
-			(at 0 0 0)
-			(layer "F.SilkS")
-			(hide yes)
-			(effects
-				(font
-					(size 1 1)
-					(thickness 0.15)
-				)
-			)
-		)
-		(property ki_fp_filters "C_*")
-		(sheetname "/")
-		(sheetfile "Engine_monitor_V1.kicad_sch")
-		(units
-			(unit
-				(name "A")
-				(pins "1" "2")
-			)
-		)
-		(attr smd)
-		(duplicate_pad_numbers_are_jumpers no)
-		(fp_line
-			(start -0.261252 -0.735)
-			(end 0.261252 -0.735)
-			(stroke
-				(width 0.12)
-				(type solid)
-			)
-			(layer "F.SilkS")
-		)
-		(fp_line
-			(start -0.261252 0.735)
-			(end 0.261252 0.735)
-			(stroke
-				(width 0.12)
-				(type solid)
-			)
-			(layer "F.SilkS")
-		)
-		(fp_rect
-			(start -1.7 -0.98)
-			(end 1.7 0.98)
-			(stroke
-				(width 0.05)
-				(type solid)
-			)
-			(fill no)
-			(layer "F.CrtYd")
-		)
-		(fp_rect
-			(start -1 -0.625)
-			(end 1 0.625)
-			(stroke
-				(width 0.1)
-				(type solid)
-			)
-			(fill no)
-			(layer "F.Fab")
-		)
-		(fp_text user "${REFERENCE}"
-			(at 0 0 0)
-			(layer "F.Fab")
-			(effects
-				(font
-					(size 0.5 0.5)
-					(thickness 0.08)
-				)
-			)
-		)
-		(pad "1" smd roundrect
-			(at -0.95 0)
-			(size 1 1.45)
-			(layers "F.Cu" "F.Mask" "F.Paste")
-			(roundrect_rratio 0.25)
-			(net "Net-(D10-K)")
-			(pintype "passive")
-		)
-		(pad "2" smd roundrect
-			(at 0.95 0)
-			(size 1 1.45)
-			(layers "F.Cu" "F.Mask" "F.Paste")
-			(roundrect_rratio 0.25)
-			(net "GND")
-			(pintype "passive")
-		)
-		(embedded_fonts no)
-		(model "${KICAD10_3DMODEL_DIR}/Capacitor_SMD.3dshapes/C_0805_2012Metric.step"
-			(offset
-				(xyz 0 0 0)
-			)
-			(scale
-				(xyz 1 1 1)
-			)
-			(rotate
-				(xyz 0 0 0)
-			)
-		)
-	)
 	(footprint "Adafruit MAX31856:0805-NO"
 		(layer "F.Cu")
@@
 		(embedded_fonts no)
 	)
+	(footprint "Resistor_SMD:R_0805_2012Metric"
+		(layer "F.Cu")
+		(at 97.7125 82.5 180)
+		(descr "Resistor SMD 0805 (2012 Metric), square (rectangular) end terminal, IPC-7351 nominal, (Body size source: IPC-SM-782 page 72, https://www.pcb-3d.com/wordpress/wp-content/uploads/ipc-sm-782a_amendment_1_and_2.pdf)")
+		(tags "resistor")
+		(property "Reference" "R14"
+			(at 0 -1.65 0)
+			(layer "F.SilkS")
+			(effects
+				(font
+					(size 1 1)
+					(thickness 0.15)
+				)
+			)
+		)
+		(property "Value" "220k"
+			(at 0 1.65 0)
+			(layer "F.Fab")
+			(effects
+				(font
+					(size 1 1)
+					(thickness 0.15)
+				)
+			)
+		)
+		(property "Datasheet" ""
+			(at 0 0 0)
+			(layer "F.Fab")
+			(hide yes)
+			(effects
+				(font
+					(size 1.27 1.27)
+				)
+			)
+		)
+		(property "Description" "Resistor"
+			(at 0 0 0)
+			(layer "F.Fab")
+			(hide yes)
+			(effects
+				(font
+					(size 1.27 1.27)
+				)
+			)
+		)
+		(property "KiLib_Generator" "SMD_2terminal_chip_molded"
+			(at 0 0 0)
+			(layer "F.SilkS")
+			(hide yes)
+			(effects
+				(font
+					(size 1 1)
+					(thickness 0.15)
+				)
+			)
+		)
+		(property ki_fp_filters "R_*")
+		(sheetname "/")
+		(sheetfile "Engine_monitor_V1.kicad_sch")
+		(units
+			(unit
+				(name "A")
+				(pins "1" "2")
+			)
+		)
+		(attr smd)
+		(duplicate_pad_numbers_are_jumpers no)
+		(fp_line
+			(start -0.227064 0.735)
+			(end 0.227064 0.735)
+			(stroke
+				(width 0.12)
+				(type solid)
+			)
+			(layer "F.SilkS")
+		)
+		(fp_line
+			(start -0.227064 -0.735)
+			(end 0.227064 -0.735)
+			(stroke
+				(width 0.12)
+				(type solid)
+			)
+			(layer "F.SilkS")
+		)
+		(fp_rect
+			(start -1.68 -0.95)
+			(end 1.68 0.95)
+			(stroke
+				(width 0.05)
+				(type solid)
+			)
+			(fill no)
+			(layer "F.CrtYd")
+		)
+		(fp_rect
+			(start -1 -0.625)
+			(end 1 0.625)
+			(stroke
+				(width 0.1)
+				(type solid)
+			)
+			(fill no)
+			(layer "F.Fab")
+		)
+		(fp_text user "${REFERENCE}"
+			(at 0 0 0)
+			(layer "F.Fab")
+			(effects
+				(font
+					(size 0.5 0.5)
+					(thickness 0.08)
+				)
+			)
+		)
+		(pad "1" smd roundrect
+			(at -0.9125 0 180)
+			(size 1.025 1.4)
+			(layers "F.Cu" "F.Mask" "F.Paste")
+			(roundrect_rratio 0.243902)
+			(net "GND")
+			(pintype "passive")
+		)
+		(pad "2" smd roundrect
+			(at 0.9125 0 180)
+			(size 1.025 1.4)
+			(layers "F.Cu" "F.Mask" "F.Paste")
+			(roundrect_rratio 0.243902)
+			(net "Net-(D10-K)")
+			(pintype "passive")
+		)
+		(embedded_fonts no)
+		(model "${KICAD10_3DMODEL_DIR}/Resistor_SMD.3dshapes/R_0805_2012Metric.step"
+			(offset
+				(xyz 0 0 0)
+			)
+			(scale
+				(xyz 1 1 1)
+			)
+			(rotate
+				(xyz 0 0 0)
+			)
+		)
+	)
 	(footprint "Package_TO_SOT_SMD:SOT-23-5"
 		(layer "F.Cu")
@@
 	)
 	(segment
+		(start 98.7 82.45)
+		(end 98.95 82.7)
+		(width 0.6)
+		(layer "F.Cu")
+		(net "GND")
+	)
+	(segment
 		(start 100.9 138.3)
 		(end 101.9 139.3)
@@
 	)
 	(segment
-		(start 90.55 94.525)
-		(end 90.55 96.225)
+		(start 98.85 79.35)
+		(end 98.85 82.275)
 		(width 0.6)
 		(layer "F.Cu")
@@
 	)
 	(segment
-		(start 98.85 79.35)
-		(end 98.85 82.3)
+		(start 90.55 94.525)
+		(end 90.55 96.225)
 		(width 0.6)
 		(layer "F.Cu")
@@
 	)
 	(segment
+		(start 98.85 82.3)
+		(end 98.7 82.45)
+		(width 0.6)
+		(layer "F.Cu")
+		(net "GND")
+	)
+	(segment
 		(start 89.2 88.6875)
 		(end 89.2 91.2)
@@
 	)
 	(segment
-		(start 99.8 138.2)
-		(end 99.9 138.3)
+		(start 98.85 82.275)
+		(end 98.625 82.5)
 		(width 0.6)
 		(layer "F.Cu")
@@
 	)
 	(segment
-		(start 98.7 82.45)
-		(end 98.95 82.7)
+		(start 99.8 138.2)
+		(end 99.9 138.3)
 		(width 0.6)
 		(layer "F.Cu")
@@
 	)
 	(segment
-		(start 98.85 82.3)
-		(end 98.7 82.45)
+		(start 98.95 82.7)
+		(end 100.6 82.7)
 		(width 0.6)
 		(layer "F.Cu")
@@
 		(net "GND")
 	)
-	(segment
-		(start 98.95 82.7)
-		(end 100.6 82.7)
-		(width 0.6)
-		(layer "F.Cu")
-		(net "GND")
-	)
 	(via
 		(at 99.9 133.5)
@@
 	)
 	(segment
-		(start 94.4 82.375)
-		(end 96.725 82.375)
+		(start 96.675 82.375)
+		(end 96.8 82.5)
 		(width 0.6)
 		(layer "F.Cu")
@@
 		(width 0.6)
 		(layer "F.Cu")
+		(net "Net-(D10-K)")
+	)
+	(segment
+		(start 94.4 82.375)
+		(end 96.675 82.375)
+		(width 0.6)
+		(layer "F.Cu")

Commit message: Trying to create a JLPCB upload files
Parts:
- R10: value 22k -> 150k
Changed lines of the file:
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@@
 			)
 		)
-		(attr through_hole)
+		(attr through_hole exclude_from_bom dnp)
 		(duplicate_pad_numbers_are_jumpers no)
 		(fp_line
@@
 			)
 		)
+		(attr exclude_from_bom dnp)
 		(duplicate_pad_numbers_are_jumpers no)
 		(fp_line
@@
 			)
 		)
-		(attr through_hole)
+		(attr through_hole exclude_from_bom dnp)
 		(duplicate_pad_numbers_are_jumpers no)
 		(fp_line
@@
 			)
 		)
-		(property "Value" "22k"
+		(property "Value" "150k"
 			(at 0 1.65 90)
 			(layer "F.Fab")
@@
 			)
 		)
-		(attr through_hole)
+		(attr through_hole exclude_from_bom dnp)
 		(duplicate_pad_numbers_are_jumpers no)
 		(fp_line
@@
 			)
 		)
-		(attr through_hole)
+		(attr through_hole exclude_from_bom dnp)
 		(duplicate_pad_numbers_are_jumpers no)
 		(fp_line
@@
 			)
 		)
+		(attr exclude_from_bom dnp)
 		(duplicate_pad_numbers_are_jumpers no)
 		(fp_line
@@
 	)
 	(segment
-		(start 88.25 88.6875)
-		(end 85.6875 88.6875)
-		(width 0.4)
-		(layer "F.Cu")
-		(net "Net-(D10-K)")
-	)
-	(segment
-		(start 96.675 82.375)
-		(end 96.8 82.5)
-		(width 0.6)
-		(layer "F.Cu")
-		(net "Net-(D10-K)")
-	)
-	(segment
-		(start 91.9 78.1)
-		(end 93.15 79.35)
-		(width 0.6)
-		(layer "F.Cu")
-		(net "Net-(D10-K)")
-	)
-	(segment
-		(start 89.2 81.9)
-		(end 89.15 81.85)
-		(width 0.4)
-		(layer "F.Cu")
-		(net "Net-(D10-K)")
-	)
-	(segment
-		(start 85.2 88.2)
-		(end 85.2 82.9)
-		(width 0.4)
-		(layer "F.Cu")
-		(net "Net-(D10-K)")
-	)
-	(segment
-		(start 85.2 82.9)
-		(end 86.2 81.9)
-		(width 0.4)
-		(layer "F.Cu")
-		(net "Net-(D10-K)")
-	)
-	(segment
-		(start 85.6875 88.6875)
-		(end 85.2 88.2)
-		(width 0.4)
-		(layer "F.Cu")
-		(net "Net-(D10-K)")
-	)
-	(segment
-		(start 90.75 80.55)
-		(end 89.15 80.55)
-		(width 0.6)
-		(layer "F.Cu")
-		(net "Net-(D10-K)")
-	)
-	(segment
-		(start 91.9 79.4)
-		(end 90.75 80.55)
-		(width 0.6)
-		(layer "F.Cu")
-		(net "Net-(D10-K)")
-	)
-	(segment
-		(start 91.9 77.75)
-		(end 91.9 78.1)
-		(width 0.6)
-		(layer "F.Cu")
-		(net "Net-(D10-K)")
-	)
-	(segment
-		(start 86.2 81.9)
-		(end 89.2 81.9)
-		(width 0.4)
-		(layer "F.Cu")
-		(net "Net-(D10-K)")
-	)
-	(segment
-		(start 93.15 79.35)
-		(end 94.4 80.6)
-		(width 0.6)
-		(layer "F.Cu")
-		(net "Net-(D10-K)")
-	)
-	(segment
-		(start 93.15 79.35)
-		(end 95.55 79.35)
-		(width 0.6)
-		(layer "F.Cu")
-		(net "Net-(D10-K)")
-	)
-	(segment
-		(start 94.4 82.375)
-		(end 96.675 82.375)
-		(width 0.6)
-		(layer "F.Cu")
-		(net "Net-(D10-K)")
-	)
-	(segment
-		(start 96.725 82.375)
-		(end 96.8 82.45)
-		(width 0.6)
-		(layer "F.Cu")
-		(net "Net-(D10-K)")
-	)
-	(segment
-		(start 91.9 77.75)
-		(end 91.9 79.4)
-		(width 0.6)
-		(layer "F.Cu")
-		(net "Net-(D10-K)")
-	)
-	(segment
-		(start 94.4 80.6)
-		(end 94.4 82.375)
-		(width 0.6)
-		(layer "F.Cu")
-		(net "Net-(D10-K)")
-	)
-	(segment
-		(start 89.15 81.85)
-		(end 89.15 80.55)
-		(width 0.4)
-		(layer "F.Cu")
-		(net "Net-(D10-K)")
-	)
-	(segment
 		(start 99.9178 130.5)
 		(end 101 130.5)
@@
 	)
 	(segment
+		(start 88.25 88.6875)
+		(end 85.6875 88.6875)
+		(width 0.4)
+		(layer "F.Cu")
+		(net "Net-(D10-K)")
+	)
+	(segment
+		(start 96.675 82.375)
+		(end 96.8 82.5)
+		(width 0.6)
+		(layer "F.Cu")
+		(net "Net-(D10-K)")
+	)
+	(segment
+		(start 91.9 78.1)
+		(end 93.15 79.35)
+		(width 0.6)
+		(layer "F.Cu")
+		(net "Net-(D10-K)")
+	)
+	(segment
+		(start 89.2 81.9)
+		(end 89.15 81.85)
+		(width 0.4)
+		(layer "F.Cu")
+		(net "Net-(D10-K)")
+	)
+	(segment
+		(start 85.2 88.2)
+		(end 85.2 82.9)
+		(width 0.4)
+		(layer "F.Cu")
+		(net "Net-(D10-K)")
+	)
+	(segment
+		(start 85.2 82.9)
+		(end 86.2 81.9)
+		(width 0.4)
+		(layer "F.Cu")
+		(net "Net-(D10-K)")
+	)
+	(segment
+		(start 85.6875 88.6875)
+		(end 85.2 88.2)
+		(width 0.4)
+		(layer "F.Cu")
+		(net "Net-(D10-K)")
+	)
+	(segment
+		(start 90.75 80.55)
+		(end 89.15 80.55)
+		(width 0.6)
+		(layer "F.Cu")
+		(net "Net-(D10-K)")
+	)
+	(segment
+		(start 91.9 79.4)
+		(end 90.75 80.55)
+		(width 0.6)
+		(layer "F.Cu")
+		(net "Net-(D10-K)")
+	)
+	(segment
+		(start 91.9 77.75)
+		(end 91.9 78.1)
+		(width 0.6)
+		(layer "F.Cu")
+		(net "Net-(D10-K)")
+	)
+	(segment
+		(start 86.2 81.9)
+		(end 89.2 81.9)
+		(width 0.4)
+		(layer "F.Cu")
+		(net "Net-(D10-K)")
+	)
+	(segment
+		(start 93.15 79.35)
+		(end 94.4 80.6)
+		(width 0.6)
+		(layer "F.Cu")
+		(net "Net-(D10-K)")
+	)
+	(segment
+		(start 93.15 79.35)
+		(end 95.55 79.35)
+		(width 0.6)
+		(layer "F.Cu")
+		(net "Net-(D10-K)")
+	)
+	(segment
+		(start 94.4 82.375)
+		(end 96.675 82.375)
+		(width 0.6)
+		(layer "F.Cu")
+		(net "Net-(D10-K)")
+	)
+	(segment
+		(start 96.725 82.375)
+		(end 96.8 82.45)
+		(width 0.6)
+		(layer "F.Cu")
+		(net "Net-(D10-K)")
+	)
+	(segment
+		(start 91.9 77.75)
+		(end 91.9 79.4)
+		(width 0.6)
+		(layer "F.Cu")
+		(net "Net-(D10-K)")
+	)
+	(segment
+		(start 94.4 80.6)
+		(end 94.4 82.375)
+		(width 0.6)
+		(layer "F.Cu")
+		(net "Net-(D10-K)")
+	)
+	(segment
+		(start 89.15 81.85)
+		(end 89.15 80.55)
+		(width 0.4)
+		(layer "F.Cu")
+		(net "Net-(D10-K)")
+	)
+	(segment
